File: devpcb/main/main.kicad_pcb (KiCad board)
At the start: 2 copper layers, 1 part, among them U1 DRV8301DCAR

Commit message: gtg sep 19 5pm
Parts:
- added C1: 100n, Capacitor_SMD:C_0402_1005Metric, F.Cu at (189.3, 117.6)
- added C10: 100n, Capacitor_SMD:C_0402_1005Metric, F.Cu at (195.0, 119.5)
- added C11: 100n, Capacitor_SMD:C_0402_1005Metric, F.Cu at (195.0, 121.5)
- added C2: 100n, Capacitor_SMD:C_0402_1005Metric, F.Cu at (189.3, 119.5)
- added C3: 100n, Capacitor_SMD:C_0402_1005Metric, F.Cu at (189.3, 121.5)
- added C4: 100n, Capacitor_SMD:C_0402_1005Metric, F.Cu at (192.2, 117.6)
- added C5: 100n, Capacitor_SMD:C_0402_1005Metric, F.Cu at (192.2, 119.5)
- added C6: 100n, Capacitor_SMD:C_0402_1005Metric, F.Cu at (192.2, 121.5)
- added C7: 1u, Capacitor_SMD:C_0603_1608Metric, F.Cu at (195.0, 107.2)
- added C8: 100n, Capacitor_SMD:C_0402_1005Metric, F.Cu at (195.0, 117.6)
- added C9: 1u, Capacitor_SMD:C_0603_1608Metric, F.Cu at (195.0, 109.7)
- added R1: 27.4, A_HDJ_Library:R_0402_1005Metric, F.Cu at (191.5, 106.9)
- added R2: 27.4, A_HDJ_Library:R_0402_1005Metric, F.Cu at (191.5, 108.9)
- added R3: 10k, A_HDJ_Library:R_0402_1005Metric, F.Cu at (191.5, 110.9)
- added R4: 10k, A_HDJ_Library:R_0402_1005Metric, F.Cu at (191.5, 112.9)
- added U2: RP2040, Package_DFN_QFN:QFN-56-1EP_7x7mm_P0.4mm_EP3.2x3.2mm, F.Cu at (183.2, 121.2)
- added U3: ~, Package_TO_SOT_THT:TO-220-3_Vertical, F.Cu at (180.2, 109.0)
Connections:
- U1 pad 10: unconnected-(U1-SDO-Pad10) -> /GPIO4
- U1 pad 11: unconnected-(U1-SCLK-Pad11) -> /GPIO2
- U1 pad 28: unconnected-(U1-AGND-Pad28) -> GND
- U1 pad 5: unconnected-(U1-*OCTW-Pad5) -> Net-(U1-*OCTW)
- U1 pad 6: unconnected-(U1-*FAULT-Pad6) -> Net-(U1-*FAULT)
- U1 pad 8: unconnected-(U1-*SCS-Pad8) -> /GPIO5
- U1 pad 9: unconnected-(U1-SDI-Pad9) -> /GPIO3

Commit message: atsr
Parts:
- added C12: 0.022µF, Capacitor_SMD:C_0402_1005Metric_Pad0.74x0.62mm_HandSolder, F.Cu at (157.9, 77.8)
- added C13: 2.2µF, Capacitor_SMD:C_0805_2012Metric, F.Cu at (156.7, 76.1)
- added C14: 1µF, Capacitor_SMD:C_0603_1608Metric, F.Cu at (157.4, 80.6)
- added C15: 1µF, Capacitor_SMD:C_0603_1608Metric, F.Cu at (157.4, 82.3)
- added C16: 4.7µF, Capacitor_SMD:C_0805_2012Metric, F.Cu at (169.7, 84.8)
- added C17: 0.1µF, Capacitor_SMD:C_0603_1608Metric, F.Cu at (172.9, 79.6)
- added C18: 0.1µF, Capacitor_SMD:C_0603_1608Metric, F.Cu at (172.9, 76.1)
- added C19: 0.1µF, Capacitor_SMD:C_0603_1608Metric, F.Cu at (172.9, 72.6)
- added C20: 10u, Capacitor_SMD:C_0805_2012Metric, F.Cu at (168.0, 34.2)
- added C21: 10u, Capacitor_SMD:C_0805_2012Metric, F.Cu at (158.2, 38.8)
- added C22: 100n, Capacitor_SMD:C_0402_1005Metric, F.Cu at (182.5, 33.0)
- added C23: 15p, Capacitor_SMD:C_0402_1005Metric, F.Cu at (174.2, 53.2)
- added C24: 15p, Capacitor_SMD:C_0402_1005Metric, F.Cu at (175.5, 53.2)
- added J1: Conn_01x03_Pin, Connector_PinHeader_2.54mm:PinHeader_1x03_P2.54mm_Vertical, F.Cu at (197.9, 69.0)
- added J2: Conn_01x03_Pin, Connector_PinHeader_2.54mm:PinHeader_1x03_P2.54mm_Vertical, F.Cu at (197.9, 77.8)
- added J3: USB_B_Micro, Connector_USB:USB_Micro-AB_Molex_47590-0001, F.Cu at (176.8, 27.1)
- added J4: Conn_01x02_Pin, Connector_PinHeader_2.54mm:PinHeader_1x02_P2.54mm_Vertical, F.Cu at (158.0, 41.8)
- added J5: Conn_01x02_Pin, Connector_PinHeader_2.54mm:PinHeader_1x02_P2.54mm_Vertical, F.Cu at (169.8, 31.2)
- added J6: Conn_01x02_Pin, Connector_PinHeader_2.54mm:PinHeader_1x02_P2.54mm_Vertical, F.Cu at (184.0, 30.5)
- added J7: Conn_01x02_Pin, Connector_PinHeader_2.54mm:PinHeader_1x02_P2.54mm_Vertical, F.Cu at (166.0, 40.2)
- added J8: Conn_01x20_Pin, Connector_PinHeader_2.54mm:PinHeader_1x20_P2.54mm_Vertical, F.Cu at (150.2, 30.7)
- added J9: Conn_01x20_Pin, Connector_PinHeader_2.54mm:PinHeader_1x20_P2.54mm_Vertical, F.Cu at (205.8, 78.8)
- added R10: 15, Resistor_SMD:R_0402_1005Metric, F.Cu at (188.7, 63.1)
- added R11: 15, Resistor_SMD:R_0402_1005Metric, F.Cu at (188.7, 73.6)
- added R12: 15, Resistor_SMD:R_0402_1005Metric, F.Cu at (188.7, 84.1)
- added R13: 1k, Resistor_SMD:R_0402_1005Metric, F.Cu at (169.8, 43.0)
- added R14: DNF, Resistor_SMD:R_0402_1005Metric, F.Cu at (169.0, 40.0)
- added R15: 1k, Resistor_SMD:R_0402_1005Metric, F.Cu at (177.8, 55.2)
- added R5: 15, Resistor_SMD:R_0402_1005Metric, F.Cu at (176.9, 63.1)
- added R6: 15, Resistor_SMD:R_0402_1005Metric, F.Cu at (176.9, 73.6)
- added R7: 15, Resistor_SMD:R_0402_1005Metric, F.Cu at (176.9, 84.1)
- added R8: 33k, Resistor_SMD:R_0402_1005Metric, F.Cu at (158.2, 72.1)
- added R9: 10k, Resistor_SMD:R_0402_1005Metric, F.Cu at (170.7, 69.6)
- added U10: W25Q128JVS, Package_SO:SOIC-8_5.3x5.3mm_P1.27mm, F.Cu at (176.5, 35.0)
- added U4: ~, Package_TO_SOT_THT:TO-220-3_Vertical, F.Cu at (179.7, 73.5)
- added U5: ~, Package_TO_SOT_THT:TO-220-3_Vertical, F.Cu at (179.7, 84.0)
- added U6: ~, Package_TO_SOT_THT:TO-220-3_Vertical, F.Cu at (191.4, 63.0)
- added U7: ~, Package_TO_SOT_THT:TO-220-3_Vertical, F.Cu at (191.4, 73.5)
- added U8: ~, Package_TO_SOT_THT:TO-220-3_Vertical, F.Cu at (191.4, 84.0)
- added U9: NCP1117-3.3_SOT223, Package_TO_SOT_SMD:SOT-223-3_TabPin2, F.Cu at (160.5, 34.0)
- added Y1: Crystal_GND23, Crystal:Crystal_SMD_3225-4Pin_3.2x2.5mm, F.Cu at (175.2, 56.8)
- moved C11 83.4 mm to (174.2, 40.8), turned to 90 degrees
- moved C3 81.9 mm to (175.5, 40.8), turned to 90 degrees
- moved C10 80.4 mm to (178.8, 40.8), turned to 90 degrees
- moved C6 77.0 mm to (169.8, 47.8), turned to 180 degrees
- moved C8 77.0 mm to (180.3, 42.0)
- moved C4 76.7 mm to (169.8, 44.2), turned to 180 degrees
- moved C2 75.6 mm to (182.3, 44.2)
- moved U2 74.8 mm to (176.1, 46.8)
- moved C9 72.6 mm to (170.0, 41.5), turned to 180 degrees
- moved C1 70.2 mm to (182.2, 47.8)
- moved R2 69.5 mm to (177.8, 40.8), turned to -90 degrees
- moved C5 68.7 mm to (177.2, 52.5), turned to -90 degrees
- moved R1 67.8 mm to (176.8, 40.8), turned to -90 degrees
- moved C7 58.5 mm to (182.5, 50.0)
- moved R4 53.9 mm to (158.2, 70.6), turned to -90 degrees
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Connections:
- U1 pad 13: unconnected-(U1-GVDD-Pad13) -> Net-(U1-GVDD)
- U1 pad 14: unconnected-(U1-CP1-Pad14) -> Net-(U1-CP1)
- U1 pad 15: unconnected-(U1-CP2-Pad15) -> Net-(U1-CP2)
- U1 pad 16: unconnected-(U1-EN_GATE-Pad16) -> /GPIO9
- U1 pad 17: unconnected-(U1-INH_A-Pad17) -> /GPIO6
- U1 pad 19: unconnected-(U1-INH_B-Pad19) -> /GPIO7
- U1 pad 21: unconnected-(U1-INH_C-Pad21) -> /GPIO8
- U1 pad 23: unconnected-(U1-DVDD-Pad23) -> Net-(U1-DVDD)
- U1 pad 27: unconnected-(U1-AVDD-Pad27) -> Net-(U1-AVDD)
- U1 pad 29: unconnected-(U1-PVDD1-Pad29) -> +12V
- U1 pad 34: unconnected-(U1-SL_C-Pad34) -> GND
- U1 pad 35: unconnected-(U1-GL_C-Pad35) -> Net-(U1-GL_C)
- U1 pad 36: unconnected-(U1-SH_C-Pad36) -> Net-(J2-Pin_3)
- U1 pad 37: unconnected-(U1-GH_C-Pad37) -> Net-(U1-GH_C)
- U1 pad 38: unconnected-(U1-BST_C-Pad38) -> Net-(U1-BST_C)
- U1 pad 39: unconnected-(U1-SL_B-Pad39) -> GND
- U1 pad 40: unconnected-(U1-GL_B-Pad40) -> Net-(U1-GL_B)
- U1 pad 41: unconnected-(U1-SH_B-Pad41) -> Net-(J2-Pin_2)
- U1 pad 42: unconnected-(U1-GH_B-Pad42) -> Net-(U1-GH_B)
- U1 pad 43: unconnected-(U1-BST_B-Pad43) -> Net-(U1-BST_B)
- U1 pad 44: unconnected-(U1-SL_A-Pad44) -> GND
- U1 pad 45: unconnected-(U1-GL_A-Pad45) -> Net-(U1-GL_A)
- U1 pad 46: unconnected-(U1-SH_A-Pad46) -> Net-(J2-Pin_1)
- U1 pad 47: unconnected-(U1-GH_A-Pad47) -> Net-(U1-GH_A)
- U1 pad 48: unconnected-(U1-BST_A-Pad48) -> Net-(U1-BST_A)
- U1 pad 49: unconnected-(U1-VDD_SPI-Pad49) -> +3V3
- U1 pad 55: unconnected-(U1-EN_BUCK-Pad55) -> Net-(U1-EN_BUCK)
- U1 pad 57: unconnected-(U1-EPAD-Pad57) -> GND
- U1 pad 7: unconnected-(U1-DTC-Pad7) -> Net-(U1-DTC)
- U3 pad 1: unconnected-(U3-Gate-Pad1) -> Net-(U3-Gate)
- U3 pad 2: unconnected-(U3-Drain-Pad2) -> Net-(J1-Pin_1)
- U3 pad 3: unconnected-(U3-Source-Pad3) -> GND
Routing:
- net +12V: track 0.00 -> 120.6 mm, vias 0 -> 12
- net Net-(J2-Pin_1): track 0.00 -> 37.8 mm, vias 0 -> 2
- net Net-(J2-Pin_3): track 0.00 -> 36.3 mm, vias 0 -> 2
- net Net-(J2-Pin_2): track 0.00 -> 33.3 mm, vias 0 -> 2
- net Net-(U1-GH_A): track 0.00 -> 30.3 mm
- net Net-(U1-GH_B): track 0.00 -> 25.0 mm, vias 0 -> 2
- net Net-(U1-GH_C): track 0.00 -> 24.1 mm, vias 0 -> 2
- net /QSPI_SS: track 0.00 -> 23.9 mm
- net Net-(J1-Pin_3): track 0.00 -> 23.6 mm
- net Net-(J1-Pin_1): track 0.00 -> 20.2 mm
- net Net-(J1-Pin_2): track 0.00 -> 20.1 mm
- net +3V3: track 0.00 -> 20.0 mm
- net /USB_D-: track 0.00 -> 17.8 mm
- net /USB_D+: track 0.00 -> 17.8 mm
- net Net-(U1-GL_A): track 0.00 -> 17.3 mm
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Other:
- board outline added: 7.5 x 2 mm

Commit message: a
Parts:
- moved C6 0.27 mm to (169.8, 47.5)
- moved C4 0.17 mm to (169.8, 44.0)
- turned J4 to 90 degrees
Routing:
- net +3V3: track 20.0 -> 183.1 mm, vias 0 -> 10
- net GND: track 2.76 -> 127.4 mm, vias 0 -> 46
- net /GPIO3: track 0.00 -> 84.3 mm, vias 0 -> 2
- net +12V: track 120.6 -> 194.8 mm, vias 12 -> 20
- net /GPIO7: track 0.00 -> 72.1 mm, vias 0 -> 1
- net /GPIO2: track 0.00 -> 70.8 mm, vias 0 -> 3
- net /GPIO6: track 0.00 -> 69.5 mm
- net /GPIO4: track 0.00 -> 64.2 mm, vias 0 -> 3
- net /GPIO9: track 0.00 -> 63.2 mm
- net /GPIO17: track 0.00 -> 58.8 mm
- net /GPIO8: track 0.00 -> 57.7 mm, vias 0 -> 1
- net /GPIO5: track 0.00 -> 56.9 mm, vias 0 -> 3
- net /GPIO18: track 0.00 -> 45.5 mm, vias 0 -> 2
- net /GPIO16: track 0.00 -> 44.9 mm
- net /GPIO19: track 0.00 -> 44.8 mm, vias 0 -> 2
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- added copper zone on B.Cu, net GND
Other:
- board size 7.5 x 2 mm -> 60 x 66.5 mm
