File: devpcb/main/main.kicad_sch (KiCad schematic)
At the start: 0 parts

Commit message: 7 51 sept 16
Parts:
- added C1, C10, C11, C2, C3, C4, C5, C6, C8: 100n, Capacitor_SMD:C_0402_1005Metric, symbol Device:C
- added C7, C9: 1u, Capacitor_SMD:C_0603_1608Metric, symbol Device:C
- added R1, R2: 27.4, A_HDJ_Library:R_0402_1005Metric, symbol Device:R
- added U1: DRV8301DCAR, DCA56_6P35X3P61, symbol DRV8301DCAR:DRV8301DCAR
- added U2: RP2040, Package_DFN_QFN:QFN-56-1EP_7x7mm_P0.4mm_EP3.2x3.2mm, symbol MCU_RaspberryPi:RP2040
Connections:
- new net: R1.2, U2.47 (USB_DP)
- new net: R2.2, U2.46 (USB_DM)
- new net +1V1: C10.1, C11.1, C9.1, U2.23 (DVDD), U2.45 (VREG_VOUT), U2.50 (DVDD)
- new net +3V3: C1.1, C2.1, C3.1, C4.1, C5.1, C6.1, C7.1, C8.1, U2.1 (IOVDD), U2.10 (IOVDD), U2.22 (IOVDD), U2.33 (IOVDD), U2.42 (IOVDD), U2.43 (ADC_AVDD), U2.49 (IOVDD)
- new net GND: C1.2, C10.2, C11.2, C2.2, C3.2, C4.2, C5.2, C6.2, C7.2, C8.2, C9.2, U2.57 (GND)
- new net GPIO0: U2.2 (GPIO0)
- new net GPIO1: U2.3 (GPIO1)
- new net GPIO10: U2.13 (GPIO10)
- new net GPIO11: U2.14 (GPIO11)
- new net GPIO12: U2.15 (GPIO12)
- new net GPIO13: U2.16 (GPIO13)
- new net GPIO14: U2.17 (GPIO14)
- new net GPIO15: U2.18 (GPIO15)
- new net GPIO16: U2.27 (GPIO16)
- new net GPIO17: U2.28 (GPIO17)
- new net GPIO18: U2.29 (GPIO18)
- new net GPIO19: U2.30 (GPIO19)
- new net GPIO2: U2.4 (GPIO2)
- new net GPIO20: U2.31 (GPIO20)
- new net GPIO21: U2.32 (GPIO21)
- new net GPIO22: U2.34 (GPIO22)
- new net GPIO23: U2.35 (GPIO23)
- new net GPIO24: U2.36 (GPIO24)
- new net GPIO25: U2.37 (GPIO25)
- new net GPIO26_ADC0: U2.38 (GPIO26_ADC0)
- new net GPIO26_ADC1: U2.39 (GPIO27_ADC1)
- new net GPIO26_ADC2: U2.40 (GPIO28_ADC2)
- new net GPIO26_ADC3: U2.41 (GPIO29_ADC3)
- new net GPIO3: U2.5 (GPIO3)
- new net GPIO4: U2.6 (GPIO4)
- new net GPIO5: U2.7 (GPIO5)
- new net GPIO6: U2.8 (GPIO6)
- new net GPIO7: U2.9 (GPIO7)
- new net GPIO8: U2.11 (GPIO8)
- new net GPIO9: U2.12 (GPIO9)
- new net USB_D+: R1.1
- new net USB_D-: R2.1
Other:
- note added: "Make sure C7 is close to pin 44 of the rp2040"
- note added: "Make sure c8 is close to pin 43"
- note added: "Make sure c9 is close to pin 45 of rp2040"

Commit message: sep 18  gn
Parts:
- added R3, R4: 10k, A_HDJ_Library:R_0402_1005Metric, symbol Device:R
Connections:
- net +3V3: now also R3.1, R4.1
- net GND: now also U1.28 (AGND)
- net GPIO2: now also U1.11 (SCLK)
- net GPIO3: now also U1.9 (SDI)
- net GPIO4: now also U1.10 (SDO)
- net GPIO5: now also U1.8 (*SCS)
- net TESTEN: now reaches U2.19 (TESTEN)
- net XIN: now reaches U2.20 (XIN)
- net XOUT: now reaches U2.21 (XOUT)
- net SWCLK: now reaches U2.24 (SWCLK)
- net SWD: now reaches U2.25 (SWD)
- net RUN: now reaches U2.26 (RUN)
- net QSPI_SD3: now reaches U2.51 (QSPI_SD3)
- net QSPI_SCLK: now reaches U2.52 (QSPI_SCLK)
- net QSPI_SD0: now reaches U2.53 (QSPI_SD0)
- net QSPI_SD2: now reaches U2.54 (QSPI_SD2)
- net QSPI_SD1: now reaches U2.55 (QSPI_SD1)
- net QSPI_SS: now reaches U2.56 (QSPI_SS)
- net at U1.5 (*OCTW): now also R3.2
- net at U1.6 (*FAULT): now also R4.2
Other:
- note added: "MISO"
- note added: "MOSI"
- moved on the sheet: C1, C10, C11, C2, C3, C4, C5, C6, C7, C8, C9, R1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

Commit message: gtg sep 19 5pm
Parts:
- added U3, U4, U5: ~, Package_TO_SOT_THT:TO-220-3_Vertical, symbol RS100N135T:RS100N135T
- U1: footprint DCA56_6P35X3P61 -> DRV8301DCAR:DCA56_6P35X3P61
Other:
- moved on the sheet: R3, R4, U1

Commit message: a
Parts:
- added C12: 0.022µF, Capacitor_SMD:C_0402_1005Metric_Pad0.74x0.62mm_HandSolder, symbol Device:C
- added C13: 2.2µF, Capacitor_SMD:C_0805_2012Metric, symbol Device:C
- added C14, C15: 1µF, Capacitor_SMD:C_0603_1608Metric, symbol Device:C
- added C16: 4.7µF, Capacitor_SMD:C_0805_2012Metric, symbol Device:C
- added C17, C18, C19: 0.1µF, Capacitor_SMD:C_0603_1608Metric, symbol Device:C
- added J1, J2: Conn_01x03_Pin, Connector_PinHeader_2.54mm:PinHeader_1x03_P2.54mm_Vertical, symbol Connector:Conn_01x03_Pin
- added R10, R11, R12, R5, R6, R7: 15, Resistor_SMD:R_0402_1005Metric, symbol Device:R
- added R8: 33k, Resistor_SMD:R_0402_1005Metric, symbol Device:R
- added R9: 10k, Resistor_SMD:R_0402_1005Metric, symbol Device:R
- added U6, U7, U8: ~, Package_TO_SOT_THT:TO-220-3_Vertical, symbol RS100N135T:RS100N135T
Connections:
- net +3V3: now also U1.49 (VDD_SPI)
- net GND: now also U1.34 (SL_C), U1.39 (SL_B), U1.44 (SL_A), U1.57 (EPAD), U3.3 (Source), U4.3 (Source), U5.3 (Source), C13.1, C14.1, C15.1, C16.2, R8.1, R9.2
- net GPIO6: now also U1.17 (INH_A)
- net GPIO7: now also U1.19 (INH_B)
- net GPIO8: now also U1.21 (INH_C)
- net GPIO9: now also U1.16 (EN_GATE)
- net at U5.1 (Gate): now also R7.2
- net at U5.2 (Drain): now also J1.3 (Pin_3)
- net at U3.1 (Gate): now also R5.2
- net at U3.2 (Drain): now also J1.1 (Pin_1)
- net at U4.1 (Gate): now also R6.2
- net at U4.2 (Drain): now also J1.2 (Pin_2)
- net at U1.13 (GVDD): now also C13.2
- net at U1.14 (CP1): now also C12.2
- net at U1.15 (CP2): now also C12.1
- net at U1.23 (DVDD): now also C14.2
- net at U1.27 (AVDD): now also C15.2
- net at U1.29 (PVDD1): now also C16.1
- net at U1.35 (GL_C): now also R7.1
- net at U1.36 (SH_C): now also C17.2, J2.3 (Pin_3), U8.3 (Source)
- net at U1.37 (GH_C): now also R12.1
- net at U1.38 (BST_C): now also C17.1
- net at U1.40 (GL_B): now also R6.1
- net at U1.41 (SH_B): now also C18.2, J2.2 (Pin_2), U7.3 (Source)
- net at U1.42 (GH_B): now also R11.1
- net at U1.43 (BST_B): now also C18.1
- net at U1.45 (GL_A): now also R5.1
- net at U1.46 (SH_A): now also C19.2, J2.1 (Pin_1), U6.3 (Source)
- net at U1.47 (GH_A): now also R10.1
- net at U1.48 (BST_A): now also C19.1
- net at U1.55 (EN_BUCK): now also R9.1
- net at U1.7 (DTC): now also R8.2
- new net: R10.2, U6.1 (Gate)
- new net: R11.2, U7.1 (Gate)
- new net: R12.2, U8.1 (Gate)
- new net +12V: U6.2 (Drain), U7.2 (Drain), U8.2 (Drain)
- no-connect marks 0 -> 21
Other:
- note added: "12v must get to the drv"
- note added: "Pull down to disable buck converter"

Commit message: atsr
Parts:
- added C20, C21: 10u, Capacitor_SMD:C_0805_2012Metric, symbol Device:C
- added C22: 100n, Capacitor_SMD:C_0402_1005Metric, symbol Device:C
- added C23, C24: 15p, Capacitor_SMD:C_0402_1005Metric, symbol Device:C
- added J3: USB_B_Micro, Connector_USB:USB_Micro-AB_Molex_47590-0001, symbol Connector:USB_B_Micro
- added J4, J5, J6, J7: Conn_01x02_Pin, Connector_PinHeader_2.54mm:PinHeader_1x02_P2.54mm_Vertical, symbol Connector:Conn_01x02_Pin
- added J8, J9: Conn_01x20_Pin, Connector_PinHeader_2.54mm:PinHeader_1x20_P2.54mm_Vertical, symbol Connector:Conn_01x20_Pin
- added R13, R15: 1k, Resistor_SMD:R_0402_1005Metric, symbol Device:R
- added R14: DNF, Resistor_SMD:R_0402_1005Metric, symbol Device:R
- added U10: W25Q128JVS, Package_SO:SOIC-8_5.3x5.3mm_P1.27mm, symbol Memory_Flash:W25Q128JVS
- added U9: NCP1117-3.3_SOT223, Package_TO_SOT_SMD:SOT-223-3_TabPin2, symbol Regulator_Linear:NCP1117-3.3_SOT223
- added Y1: Crystal_GND23, Crystal:Crystal_SMD_3225-4Pin_3.2x2.5mm, symbol Device:Crystal_GND23
Connections:
- net +12V: now also C16.1, U1.29 (PVDD1), J9.12 (Pin_12), J9.13 (Pin_13), J9.14 (Pin_14), J9.15 (Pin_15)
- net +3V3: now also C22.1, J4.2 (Pin_2), J8.1 (Pin_1), R14.2, U10.8 (VCC)
- net GND: now also C20.2, C21.2, C22.2, C23.1, C24.1, J3.5 (GND), J3.6 (Shield), J6.1 (Pin_1), J6.2 (Pin_2), J7.1 (Pin_1), J9.17 (Pin_17), J9.18 (Pin_18), J9.19 (Pin_19), J9.20 (Pin_20), U10.4 (GND), U9.1 (GND), Y1.2, Y1.3
- net GPIO0: now also J8.2 (Pin_2)
- net GPIO1: now also J8.3 (Pin_3)
- net GPIO10: now also J8.12 (Pin_12)
- net GPIO11: now also J8.13 (Pin_13)
- net GPIO12: now also J8.14 (Pin_14)
- net GPIO13: now also J8.15 (Pin_15)
- net GPIO14: now also J8.16 (Pin_16)
- net GPIO15: now also J8.17 (Pin_17)
- net GPIO16: now also J8.18 (Pin_18)
- net GPIO17: now also J8.19 (Pin_19)
- net GPIO18: now also J8.20 (Pin_20)
- net GPIO19: now also J9.1 (Pin_1)
- net GPIO2: now also J8.4 (Pin_4)
- net GPIO20: now also J9.2 (Pin_2)
- net GPIO21: now also J9.3 (Pin_3)
- net GPIO22: now also J9.4 (Pin_4)
- net GPIO23: now also J9.5 (Pin_5)
- net GPIO24: now also J9.6 (Pin_6)
- net GPIO25: now also J9.7 (Pin_7)
- net GPIO26_ADC0: now also J9.8 (Pin_8)
- net GPIO26_ADC1: now also J9.9 (Pin_9)
- net GPIO26_ADC2: now also J9.10 (Pin_10)
- net GPIO26_ADC3: now also J9.11 (Pin_11)
- net GPIO3: now also J8.5 (Pin_5)
- net GPIO4: now also J8.6 (Pin_6)
- net GPIO5: now also J8.7 (Pin_7)
- net GPIO6: now also J8.8 (Pin_8)
- net GPIO7: now also J8.9 (Pin_9)
- net GPIO8: now also J8.10 (Pin_10)
- net GPIO9: now also J8.11 (Pin_11)
- net QSPI_SCLK: now also U10.6 (CLK)
- net QSPI_SD0: now also U10.5 (DI/IO_{0})
- net QSPI_SD1: now also U10.2 (DO/IO_{1})
- net QSPI_SD2: now also U10.3 (~{WP}/IO_{2})
- net QSPI_SD3: now also U10.7 (~{HOLD}/~{RESET}/IO_{3})
- net QSPI_SS: now also R13.2, R14.1, U10.1 (~{CS})
- net USB_D+: now also J3.3 (D+)
- net USB_D-: now also J3.2 (D-)
- net XIN: now also C23.2, Y1.1
- net XOUT: now also R15.2
- new net: C21.1, J4.1 (Pin_1), U9.2 (VO)
- new net: C24.2, R15.1, Y1.4
- new net: J3.1 (VBUS), J5.1 (Pin_1)
- new net USB_BOOT: J7.2 (Pin_2), R13.1
- new net VBUS: C20.1, J5.2 (Pin_2), U9.3 (VI)
- no-connect marks 21 -> 23
Other:
- note added: "Gnd pins"
- note added: "Use usb 5v or external"
- note added: "allow to use or not use external 3v3 power"

Commit message: af
Other:
- note added: "CRYSTAL"
- note added: "GATE DRIVER"
- note added: "RP2040"
- note added: "SPI FLASH"
- note added: "USB AND POWER"
Changed lines of the file:
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@@
 	(generator_version "9.0")
 	(paper "A2")
+	(rectangle
+		(start 15.24 160.02)
+		(end 133.35 203.2)
+		(stroke
+			(width 0)
+			(type default)
+		)
+		(fill
+			(type none)
+		)
+	)
+	(rectangle
+		(start 15.24 274.32)
+		(end 68.58 303.53)
+		(stroke
+			(width 0)
+			(type default)
+		)
+		(fill
+			(type none)
+		)
+	)
+	(rectangle
+		(start 204.47 40.64)
+		(end 402.59 146.05)
+		(stroke
+			(width 0)
+			(type default)
+		)
+		(fill
+			(type none)
+		)
+	)
+	(rectangle
+		(start 11.43 13.97)
+		(end 191.77 148.59)
+		(stroke
+			(width 0)
+			(type default)
+		)
+		(fill
+			(type none)
+		)
+	)
+	(rectangle
+		(start 15.24 213.36)
+		(end 95.25 265.43)
+		(stroke
+			(width 0)
+			(type default)
+		)
+		(fill
+			(type none)
+		)
+	)
 	(text "allow to use or not use\nexternal 3v3 power"
 		(exclude_from_sim no)
@@
 		)
 	)
+	(text "SPI FLASH\n"
+		(exclude_from_sim no)
+		(at 34.544 269.24 0)
+		(effects
+			(font
+				(size 2.54 2.54)
+			)
+		)
+	)
 	(text "12v must get to the drv"
 		(exclude_from_sim no)
@@
 			(font
 				(size 1.27 1.27)
+			)
+		)
+	)
+	(text "GATE DRIVER\n"
+		(exclude_from_sim no)
+		(at 218.948 152.654 0)
+		(effects
+			(font
+				(size 2.54 2.54)
+			)
+		)
+	)
+	(text "USB AND POWER"
+		(exclude_from_sim no)
+		(at 32.258 207.01 0)
+		(effects
+			(font
+				(size 2.54 2.54)
+			)
+		)
+	)
+	(text "CRYSTAL\n"
+		(exclude_from_sim no)
+		(at 34.036 309.118 0)
+		(effects
+			(font
+				(size 2.54 2.54)
 			)
 		)
@@
 			)
 		)
+	)
+	(text "RP2040\n\n"
+		(exclude_from_sim no)
+		(at 23.368 154.686 0)
+		(effects
+			(font
+				(size 2.54 2.54)
+			)
+		)
